File: kicad/jspi1_rpi/jspi1_rpi.kicad_pcb (KiCad board)
At the start: 2 copper layers, 109 x 64 mm, 9 parts, among them J1 Raspberry_Pi_2_3, J2 Conn_02x20_Odd_Even, J3 Conn_02x10_Odd_Even, J4 Conn_02x10_Odd_Even, J5 Conn_02x06_Odd_Even, U1 TXS0108EPW, U2 AMS1117-1.8

Commit message: routed pcb
Parts:
- J3, J4: footprint Connector_PinSocket_2.54mm:PinSocket_2x10_P2.54mm_Vertical -> Connector_IDC:IDC-Header_2x10_P2.54mm_Vertical
- moved J5 11.4 mm to (277.2, 23.9), turned to 90 degrees
- moved J3 5.24 mm to (223.6, 32.2)
- moved J4 2.06 mm to (259.6, 24.0)
Routing:
- net Net-(J4-Pad1): track 6.00 -> 20.9 mm, vias 0 -> 1
- net /T_VCC2: track 12.1 -> 24.7 mm
- net Net-(J4-Pad2): track 6.22 -> 18.5 mm, vias 0 -> 1
- net Net-(J4-Pad12): track 31.4 -> 21.2 mm
- net Net-(J4-Pad3): track 11.5 -> 20.6 mm, vias 0 -> 1
- net Net-(J4-Pad4): track 11.7 -> 20.7 mm, vias 0 -> 1
- net Net-(J4-Pad11): track 31.2 -> 22.6 mm, vias 0 -> 1
- net Net-(J2-Pad24): track 26.6 -> 20.1 mm, vias 2 -> 0
- net GND: track 164.6 -> 171.0 mm, vias 4 -> 6
- net Net-(J4-Pad5): track 16.4 -> 22.0 mm, vias 0 -> 1
- net /T_VCC1: track 56.9 -> 62.3 mm
- net Net-(J4-Pad6): track 16.6 -> 22.1 mm
- net Net-(J4-Pad9): track 26.3 -> 21.9 mm, vias 0 -> 1
- net Net-(J2-Pad22): track 25.1 -> 20.9 mm, vias 2 -> 0
- net Net-(J4-Pad10): track 26.5 -> 23.4 mm
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- added copper zone on B.Cu, net GND
- added copper zone on F.Cu, net GND
Other:
- board size 109 x 64 mm -> 109 x 60 mm
- board text added: "1.8V"
- board text added: "3.3V"

Commit message: Order v1
Parts:
- added C1: 100n, Capacitor_SMD:C_0805_2012Metric_Pad1.18x1.45mm_HandSolder, F.Cu at (196.0, 51.0)
- added C2: 1uF, Capacitor_SMD:C_0805_2012Metric_Pad1.18x1.45mm_HandSolder, F.Cu at (195.0, 23.0)
- added C3: 1uF, Capacitor_SMD:C_0805_2012Metric_Pad1.18x1.45mm_HandSolder, F.Cu at (200.0, 23.0)
- added C4: 100n, Capacitor_SMD:C_0805_2012Metric_Pad1.18x1.45mm_HandSolder, F.Cu at (200.0, 51.0)
- moved J1 11.0 mm to (185.9, 27.2)
- moved U1 8.24 mm to (198.2, 43.8)
- moved U2 5.68 mm to (195.7, 29.5)
- moved J2 4.08 mm to (207.1, 26.9)
- moved J5 0.89 mm to (276.4, 23.9)
- moved J4 0.47 mm to (259.1, 24.0)
Connections:
- net Net-(J1-Pad1) renamed +3V3
- J4 pad 16: (no net) -> /T_MOSI
- J4 pad 18: (no net) -> /T_CLK
- J4 pad 20: (no net) -> /T_MISO
- U1 pad 11: (no net) -> GND
Routing:
- net GND: track 171.0 -> 190.4 mm, vias 6 -> 2
- net /T_MOSI: track 59.0 -> 77.8 mm, vias 1 -> 2
- net /T_MISO: track 20.2 -> 35.8 mm
- net /T_CLK: track 48.2 -> 63.7 mm, vias 2 -> 1
- net /T_VCC1: track 62.3 -> 71.1 mm, vias 2 -> 4
- net Net-(J1-Pad3): track 28.9 -> 35.3 mm, vias 2 -> 0
- net Net-(J1-Pad8): track 16.2 -> 9.90 mm, vias 2 -> 0
- net Net-(J2-Pad13): track 25.1 -> 19.0 mm, vias 2 -> 3
- net Net-(J2-Pad26): track 26.5 -> 20.6 mm, vias 1 -> 0
- net Net-(J2-Pad9): track 16.4 -> 10.7 mm
- net Net-(J2-Pad11): track 12.7 -> 7.02 mm, vias 2 -> 0
- net Net-(J2-Pad20): track 23.6 -> 18.5 mm, vias 1 -> 0
- net Net-(J2-Pad22): track 20.9 -> 16.0 mm
- net Net-(J1-Pad10): track 13.8 -> 8.85 mm, vias 2 -> 0
- net /T_GND: track 20.9 -> 16.2 mm
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Other:
- board size 109 x 60 mm -> 97 x 60 mm
- board text added: "JLCJLCJLCJLC"
- board text added: "MSI JSPI1 to RPi Adapter for 1.8V"
